Commit message: modification

File: src/robot_gazebo_ros2_control/urdf/robot_8leg.urdf (robot description, URDF)
Before this commit: robot robot, 35 links, 34 joints
Links:
- removed link conct0
- added link conct0a, mass 0.05; collision cylinder length=0.04 radius=0.06; visual cylinder length=0.04 radius=0.06
- added link conct0b, mass 0.05; collision cylinder length=0.04 radius=0.06; visual cylinder length=0.04 radius=0.06
Joints:
- added joint torso: type continuous, parent conct0b, child conct0a, origin xyz=0.04 0 0, axis 0 1 0
- joint Torso00: origin xyz=0.08 0 0 -> xyz=0.04 0 0; parent conct0 -> conct0a
- joint Torso01: child conct0 -> conct0b
